File: KICad_Project/Gruzik2.0/Gruzik2.0.kicad_sch (KiCad schematic)
At the start: 46 parts, among them U1 STM32F103C8T6, U2 LM1117MP-3.3, U3 LM1117MP-5.0, U3V40F7-POLOLU1 Conn_01x06, U3V40F7-POLOLU2 Conn_01x06, U4 TB6612FNG, U5 TB6612FNG, Y1 8MHz

Commit message: 0.1
Parts:
- renumbered Line_Sensor1 to Line_Sensor
Changed lines of the file:
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@@
   (symbol (lib_id "Connector_Generic:Conn_01x11") (at 147.32 36.83 0) (unit 1)
     (in_bom yes) (on_board yes) (dnp no) (fields_autoplaced)
-    (property "Reference" "Line_Sensor1" (at 149.86 36.195 0)
+    (property "Reference" "Line_Sensor" (at 149.86 36.195 0)
       (effects (font (size 1.27 1.27)) (justify left))
     )
@@
       (project "Gruzik2.0"
         (path "/8a909c0c-17f2-41d1-a010-8c6165729605"
-          (reference "Line_Sensor1") (unit 1)
+          (reference "Line_Sensor") (unit 1)
         )
       )

Commit message: 0.2
Parts:
- removed Line_Sensor: Conn_01x11, Connector_FFC-FPC:Molex_200528-0110_1x11-1MP_P1.00mm_Horizontal, symbol Connector_Generic:Conn_01x11
- removed UART-HC-5: Conn_01x06, Connector_PinSocket_2.54mm:PinSocket_1x06_P2.54mm_Vertical, symbol Connector_Generic:Conn_01x06
- added GRUZIK2.0: Conn_01x15, Connector_FFC-FPC:Molex_200528-0150_1x15-1MP_P1.00mm_Horizontal, symbol Connector_Generic:Conn_01x15
- added U7: HC-05, HC-05_module:XCVR_HC-05, symbol HC-05:HC-05
- C10, C11, C12, C13, C2, C3, C4, C5, C6, C7, C8, C9: footprint Capacitor_SMD:C_0402_1005Metric -> Capacitor_SMD:C_0603_1608Metric
- L1: footprint Inductor_SMD:L_0402_1005Metric -> Inductor_SMD:L_0603_1608Metric
- R1: footprint Resistor_SMD:R_0402_1005Metric -> Resistor_SMD:R_0603_1608Metric
- renumbered Motor-Battery1 to Motor-Battery_L1, Motor-Battery2 to Motor-Battery_R1
Connections:
- net +3.3V: now also U7.12 (3.3_VCC)
- net +5V: now also GRUZIK2.0.1 (Pin_1), GRUZIK2.0.2 (Pin_2), GRUZIK2.0.3 (Pin_3)
- net GND: now also GRUZIK2.0.13 (Pin_13), GRUZIK2.0.14 (Pin_14), GRUZIK2.0.15 (Pin_15), U7.13 (GND), U7.21 (GND), U7.22 (GND)
- net PA0: now also GRUZIK2.0.4 (Pin_4)
- net PA1: now also GRUZIK2.0.5 (Pin_5)
- net PA2: now also GRUZIK2.0.6 (Pin_6)
- net PA3: now also GRUZIK2.0.7 (Pin_7)
- net PA4: now also GRUZIK2.0.8 (Pin_8)
- net PA5: now also GRUZIK2.0.9 (Pin_9)
- net PA6: now also GRUZIK2.0.10 (Pin_10)
- net PA7: now also GRUZIK2.0.11 (Pin_11)
- net PB0: now also GRUZIK2.0.12 (Pin_12)
- net PB10: now also U7.2 (UART-RX)
- net PB11: now also U7.1 (UART-TX)
- no-connect marks 4 -> 2
Other:
- note added: "HC-05 Bluetooth module"
- note added: "TODO: footprint of polarized capacitors / figure out how to mount cleaners for wheels"
- note removed: "Nie tym razem Uarcie !! Tym razem bedzie dobrze Rx-Tx-SreX"
- note removed: "Rx - Tx"
- note removed: "Tx - Rx"
- note removed: "UART1 - HC-05"
- moved on the sheet: C14, C15, C16, C17, C18, C19, Motor-Battery_L1, Motor-Battery_R1, Motor-STAB-Battery-L1, Motor-STAB-Battery-R1, Motor_L1, Motor_R1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

Commit message: 0.3
Parts:
- removed GRUZIK2.0: Conn_01x15, Connector_FFC-FPC:Molex_200528-0150_1x15-1MP_P1.00mm_Horizontal, symbol Connector_Generic:Conn_01x15
- added GRUZIK2.0: Conn_01x16, Connector_FFC-FPC:Molex_200528-0160_1x16-1MP_P1.00mm_Horizontal, symbol Connector_Generic:Conn_01x16
- renumbered Motor_R1 to MOTOR_L, Motor_L1 to MOTOR_L, SW_Reset1 to RESET, UART-USB1 to UART, Vin-Battery1 to VIN
Connections:
- net +5V: now also GRUZIK2.0.2 (Pin_2), GRUZIK2.0.3 (Pin_3), GRUZIK2.0.4 (Pin_4)
- net GND: now also U4.10 (PGND2), U4.3 (PGND1), U4.4 (PGND1), U4.9 (PGND2), U5.10 (PGND2), U5.3 (PGND1), U5.4 (PGND1), U5.9 (PGND2), GRUZIK2.0.14 (Pin_14), GRUZIK2.0.15 (Pin_15), GRUZIK2.0.16 (Pin_16)
- net PA0: now also GRUZIK2.0.5 (Pin_5)
- net PA1: now also GRUZIK2.0.6 (Pin_6)
- net PA10: now also U7.1 (UART-TX)
- net PA2: now also GRUZIK2.0.7 (Pin_7)
- net PA3: now also GRUZIK2.0.8 (Pin_8)
- net PA4: now also GRUZIK2.0.9 (Pin_9)
- net PA5: now also GRUZIK2.0.10 (Pin_10)
- net PA6: now also GRUZIK2.0.11 (Pin_11)
- net PA7: now also GRUZIK2.0.12 (Pin_12)
- net PA9: now also U7.2 (UART-RX)
- net PB0: now also GRUZIK2.0.13 (Pin_13)
- net PB10: no longer U7.2 (UART-RX)
- net PB11: no longer U7.1 (UART-TX)
- no-connect marks 2 -> 3

Commit message: 0.4
Parts:
- removed PROG1: Conn_01x04_Pin, Connector_PinHeader_2.54mm:PinHeader_1x04_P2.54mm_Vertical, symbol Connector:Conn_01x04_Pin
- added C20: 100n, Capacitor_SMD:C_0603_1608Metric, symbol Device:C_Small
- added PROG1: Conn_01x05, Connector_PinHeader_2.54mm:PinHeader_1x05_P2.54mm_Vertical, symbol Connector_Generic:Conn_01x05
- renumbered MOTOR_L to MOTOR_R, RESET to RESET1, UART to UART1, VIN to VIN1
Connections:
- net +3.3V: now also C17.1, C18.1, U4.20 (VCC), U5.20 (VCC)
- net +5V: now also PROG1.5 (Pin_5); no longer C17.1, C18.1, U4.20 (VCC), U5.20 (VCC)
- net GND: now also C20.1, PROG1.1 (Pin_1)
- net SWCLK: now also PROG1.2 (Pin_2)
- net SWDIO: now also PROG1.3 (Pin_3)
- net RESET: now reaches RESET1.2 (B), U1.7 (NRST)
- net RESET: now also C20.2, PROG1.4 (Pin_4)

Commit message: 0.5
Parts:
- removed VIN1: Conn_01x03, Connector_JST:JST_XH_B3B-XH-A_1x03_P2.50mm_Vertical, symbol Connector_Generic:Conn_01x03
- added VIN1: Conn_01x02, Connector_PinSocket_2.54mm:PinSocket_1x02_P2.54mm_Vertical, symbol Connector_Generic:Conn_01x02
- renumbered MOTOR_L to MOTOR_L1, MOTOR_R to MOTOR_R1
Connections:
- net GND: now also VIN1.2 (Pin_2)
- net VDC: now also VIN1.1 (Pin_1)
Changed lines of the file:
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@@
     (stroke (width 0) (type default))
   )
-  (wire (pts (xy 142.24 69.85) (xy 147.32 69.85))
+  (wire (pts (xy 143.51 67.31) (xy 147.32 67.31))
     (stroke (width 0) (type default))
   )
@@
   (symbol (lib_id "Connector_Generic:Conn_01x02") (at 264.16 77.47 270) (unit 1)
     (in_bom yes) (on_board yes) (dnp no) (fields_autoplaced)
-    (property "Reference" "MOTOR_R" (at 266.7 76.835 90)
+    (property "Reference" "MOTOR_R1" (at 266.7 76.835 90)
       (effects (font (size 1.27 1.27)) (justify left))
     )
@@
       (project "Gruzik2.0"
         (path "/8a909c0c-17f2-41d1-a010-8c6165729605"
-          (reference "MOTOR_R") (unit 1)
+          (reference "MOTOR_R1") (unit 1)
         )
       )
@@
     )
   )
-  (symbol (lib_id "power:GND") (at 142.24 69.85 270) (unit 1)
+  (symbol (lib_id "power:GND") (at 143.51 67.31 270) (unit 1)
     (in_bom yes) (on_board yes) (dnp no) (fields_autoplaced)
-    (property "Reference" "#PWR026" (at 135.89 69.85 0)
+    (property "Reference" "#PWR026" (at 137.16 67.31 0)
       (effects (font (size 1.27 1.27)) hide)
     )
-    (property "Value" "GND" (at 138.43 70.485 90)
+    (property "Value" "GND" (at 139.7 67.945 90)
       (effects (font (size 1.27 1.27)) (justify right))
     )
-    (property "Footprint" "" (at 142.24 69.85 0)
+    (property "Footprint" "" (at 143.51 67.31 0)
       (effects (font (size 1.27 1.27)) hide)
     )
-    (property "Datasheet" "" (at 142.24 69.85 0)
+    (property "Datasheet" "" (at 143.51 67.31 0)
       (effects (font (size 1.27 1.27)) hide)
     )
@@
     )
   )
-  (symbol (lib_id "Connector_Generic:Conn_01x03") (at 152.4 67.31 0) (unit 1)
-    (in_bom yes) (on_board yes) (dnp no) (fields_autoplaced)
-    (property "Reference" "VIN1" (at 154.94 66.675 0)
-      (effects (font (size 1.27 1.27)) (justify left))
-    )
-    (property "Value" "Conn_01x03" (at 154.94 69.215 0)
-      (effects (font (size 1.27 1.27)) (justify left))
-    )
-    (property "Footprint" "Connector_JST:JST_XH_B3B-XH-A_1x03_P2.50mm_Vertical" (at 152.4 67.31 0)
-      (effects (font (size 1.27 1.27)) hide)
-    )
-    (property "Datasheet" "~" (at 152.4 67.31 0)
-      (effects (font (size 1.27 1.27)) hide)
-    )
-    (pin "1")
-    (pin "2")
-    (pin "3")
-    (instances
-      (project "Gruzik2.0"
-        (path "/8a909c0c-17f2-41d1-a010-8c6165729605"
-          (reference "VIN1") (unit 1)
-        )
-      )
-    )
-  )
   (symbol (lib_id "Driver_Motor:TB6612FNG") (at 243.84 143.51 0) (unit 1)
     (in_bom yes) (on_board yes) (dnp no) (fields_autoplaced)
@@
     )
   )
+  (symbol (lib_id "Connector_Generic:Conn_01x02") (at 152.4 64.77 0) (unit 1)
+    (in_bom yes) (on_board yes) (dnp no) (fields_autoplaced)
+    (property "Reference" "VIN1" (at 154.94 65.405 0)
+      (effects (font (size 1.27 1.27)) (justify left))
+    )
+    (property "Value" "Conn_01x02" (at 154.94 67.945 0)
+      (effects (font (size 1.27 1.27)) (justify left))
+    )
+    (property "Footprint" "Connector_PinSocket_2.54mm:PinSocket_1x02_P2.54mm_Vertical" (at 152.4 64.77 0)
+      (effects (font (size 1.27 1.27)) hide)
+    )
+    (property "Datasheet" "~" (at 152.4 64.77 0)
+      (effects (font (size 1.27 1.27)) hide)
+    )
+    (pin "1")
+    (pin "2")
+    (instances
+      (project "Gruzik2.0"
+        (path "/8a909c0c-17f2-41d1-a010-8c6165729605"
+          (reference "VIN1") (unit 1)
+        )
+      )
+    )
+  )
   (symbol (lib_id "Regulator_Linear:LM1117MP-3.3") (at 139.7 119.38 0) (unit 1)
     (in_bom yes) (on_board yes) (dnp no) (fields_autoplaced)
@@
   (symbol (lib_id "Connector_Generic:Conn_01x02") (at 264.16 160.02 270) (unit 1)
     (in_bom yes) (on_board yes) (dnp no) (fields_autoplaced)
-    (property "Reference" "MOTOR_L" (at 266.7 159.385 90)
+    (property "Reference" "MOTOR_L1" (at 266.7 159.385 90)
       (effects (font (size 1.27 1.27)) (justify left))
     )
@@
       (project "Gruzik2.0"
         (path "/8a909c0c-17f2-41d1-a010-8c6165729605"
-          (reference "MOTOR_L") (unit 1)
+          (reference "MOTOR_L1") (unit 1)
         )
       )
