File: KICad_Project/Gruzik2.0/Gruzik2.0.kicad_pcb (KiCad board)
At the start: 2 copper layers, 128 x 39.9 mm, 54 parts, among them U1 STM32F103C8T6, U2 LM1117MP-3.3, U3 LM1117MP-5.0, U3V40F7-POLOLU Conn_01x06, U4 TB6612FNG, U5 TB6612FNG, U7 HC-05, Y1 8MHz

Commit message: 0.3
Parts:
-    UART   : renamed from UART-USB
- GRUZIK2.0: value Conn_01x15 -> Conn_01x16; footprint Connector_FFC-FPC:Molex_200528-0150_1x15-1MP_P1.00mm_Horizontal -> Connector_FFC-FPC:Molex_200528-0160_1x16-1MP_P1.00mm_Horizontal; moved to B.Cu
- MOTOR L: renamed from Motor_L
- MOTOR R: renamed from Motor_R
- R1: moved to F.Cu
- moved C3 31.0 mm to (86.1, 148.7), turned to 180 degrees
- moved C5 30.6 mm to (86.6, 145.4), turned to 180 degrees
- moved Y1 28.0 mm to (87.4, 151.8)
- moved C18 8.58 mm to (118.7, 161.8), turned to 90 degrees
- moved U7 8.36 mm to (105.1, 149.0), turned to -90 degrees
- moved R2 8.24 mm to (107.2, 164.9), turned to -90 degrees
- moved R4 7.36 mm to (108.8, 164.9), turned to -90 degrees
- moved C17 6.03 mm to (116.8, 161.8), turned to 90 degrees
- moved MOTOR R 5.24 mm to (150.8, 171.0)
- moved C9 4.90 mm to (83.1, 150.7)
- moved C8 4.90 mm to (83.1, 148.9)
- moved L1 4.90 mm to (83.1, 147.1)
- moved C11 3.47 mm to (115.0, 161.8), turned to 90 degrees
- moved C15 2.10 mm to (61.1, 147.6), turned to 0 degrees
- moved C19 1.46 mm to (61.1, 145.9), turned to 0 degrees
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- renumbered Motor-Battery_L to Motor-Battery_L1, Motor-Battery_R to Motor-Battery_R1, Motor-STAB-Battery-L to Motor-STAB-Battery-L1, Motor-STAB-Battery-R to Motor-STAB-Battery-R1, SW_Reset to RESET, U3V40F7-POLOLU to U3V40F7-POLOLU1, U3V40F7-POLOLU to U3V40F7-POLOLU2, Vin-Battery to VIN
Connections:
- GRUZIK2.0 pad 1: +5V -> unconnected-(GRUZIK2.0-Pin_1-Pad1)
- GRUZIK2.0 pad 10: PA6 -> PA5
- GRUZIK2.0 pad 11: PA7 -> PA6
- GRUZIK2.0 pad 12: PB0 -> PA7
- GRUZIK2.0 pad 13: GND -> PB0
- GRUZIK2.0 pad 4: PA0 -> +5V
- GRUZIK2.0 pad 5: PA1 -> PA0
- GRUZIK2.0 pad 6: PA2 -> PA1
- GRUZIK2.0 pad 7: PA3 -> PA2
- GRUZIK2.0 pad 8: PA4 -> PA3
- GRUZIK2.0 pad 9: PA5 -> PA4
- U4 pad 10: Net-(U4-PGND1-Pad3) -> GND
- U4 pad 3: Net-(U4-PGND1-Pad3) -> GND
- U4 pad 4: Net-(U4-PGND1-Pad3) -> GND
- U4 pad 9: Net-(U4-PGND1-Pad3) -> GND
- U5 pad 10: Net-(U5-PGND1-Pad3) -> GND
- U5 pad 3: Net-(U5-PGND1-Pad3) -> GND
- U5 pad 4: Net-(U5-PGND1-Pad3) -> GND
- U5 pad 9: Net-(U5-PGND1-Pad3) -> GND
- U7 pad 1: PB11 -> PA10
- U7 pad 2: PB10 -> PA9
Routing:
- net VDC: track 0.00 -> 165.0 mm, vias 0 -> 3
- net PB6: track 0.00 -> 120.4 mm, vias 0 -> 2
- net PB9: track 0.00 -> 80.6 mm
- net PB15: track 0.00 -> 74.8 mm, vias 0 -> 4
- net PB7: track 0.00 -> 74.5 mm, vias 0 -> 2
- net GND: track 0.00 -> 70.8 mm, vias 0 -> 18
- net PB14: track 0.00 -> 68.3 mm, vias 0 -> 4
- net PB10: track 0.00 -> 67.9 mm, vias 0 -> 2
- net SWCLK: track 0.00 -> 67.7 mm, vias 0 -> 1
- net PB4: track 0.00 -> 66.1 mm
- net PB5: track 0.00 -> 66.0 mm
- net PB11: track 0.00 -> 64.6 mm, vias 0 -> 2
- net SWDIO: track 0.00 -> 61.9 mm, vias 0 -> 1
- net /BOOT0: track 0.00 -> 61.5 mm, vias 0 -> 1
- net PC13: track 0.00 -> 49.7 mm, vias 0 -> 1
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- added copper zone on In1.Cu, net +3.3V
- added copper zone on In1.Cu, net +5V
- added copper zone on In2.Cu, net +5V
- added copper zone on B.Cu, net GND
- added copper zone on F.Cu, net GND
Other:
- copper layers 2 -> 4
- board text added: "+5V"
- board text added: "GND"
- board text added: "Rx"
- board text added: "SWCLK"
- board text added: "SWDIO"
- board text added: "Tx"
- board text removed: "BATTERY"
- board text removed: "Bluetooth HC-05"

Commit message: 0.4
Parts:
- removed the PROG at (149.6, 135.5)
- added C20: 100n, Capacitor_SMD:C_0603_1608Metric, B.Cu at (82.8, 137.3)
- added PROG: Conn_01x05, Connector_PinHeader_2.54mm:PinHeader_1x05_P2.54mm_Vertical, F.Cu at (148.4, 135.6)
- UART1: renamed from    UART   
- moved D1 15.2 mm to (115.6, 134.5)
- moved R3 15.2 mm to (119.6, 134.5)
- moved C7 14.1 mm to (80.8, 158.5), turned to -90 degrees
- moved C6 11.7 mm to (82.6, 158.5), turned to -90 degrees
- moved C4 9.38 mm to (84.4, 158.5), turned to -90 degrees
- moved C2 7.21 mm to (86.1, 158.5), turned to -90 degrees
- moved C1 5.35 mm to (87.9, 158.5), turned to -90 degrees
- moved R1 1.64 mm to (144.4, 134.6)
- moved BOOT1 1.64 mm to (138.4, 135.6)
- renumbered BOOT to BOOT1, RESET to RESET1, VIN to VIN1
Connections:
- net Net-(SW_Reset1-B) renamed RESET
- C17 pad 1: +5V -> +3.3V
- C18 pad 1: +5V -> +3.3V
- U4 pad 20: +5V -> +3.3V
- U5 pad 20: +5V -> +3.3V
Routing:
- net RESET: track 39.2 -> 110.9 mm, vias 1 -> 2
- net PC13: track 49.7 -> 34.6 mm
- net +3.3V: track 45.9 -> 53.3 mm, vias 8 -> 10
- net +5V: track 38.0 -> 31.6 mm, vias 4 -> 2
- net SWCLK: track 67.7 -> 63.4 mm, vias 1 -> 2
- net /BOOT0: track 61.5 -> 59.6 mm
- net SWDIO: track 61.9 -> 63.2 mm
Other:
- board text added: "RESET"

Commit message: 0.5
Parts:
- removed VIN1: Conn_01x03, Connector_JST:JST_XH_B3B-XH-A_1x03_P2.50mm_Vertical
- added + VIN -: Conn_01x02, Connector_PinSocket_2.54mm:PinSocket_1x02_P2.54mm_Vertical, F.Cu at (133.6, 169.7)
- added G***: LOGO, SN-LAB-logo:SN-LAB, F.Cu at (63.3, 166.5)
- moved C2 22.1 mm to (104.1, 145.6), turned to 90 degrees
- moved C4 21.9 mm to (105.5, 152.7), turned to 90 degrees
- moved C1 19.3 mm to (102.3, 145.6), turned to 90 degrees
- moved D1 14.6 mm to (130.1, 135.5)
- moved R3 14.6 mm to (134.2, 135.5)
- moved C7 14.2 mm to (95.0, 158.6), turned to 0 degrees
- moved C6 12.5 mm to (95.0, 157.0), turned to 0 degrees
- moved L1 7.86 mm to (86.1, 154.4), turned to -90 degrees
- moved C9 7.51 mm to (89.6, 154.4), turned to 90 degrees
- moved C8 7.26 mm to (87.8, 154.4), turned to 90 degrees
- moved C10 1.88 mm to (130.3, 170.7), turned to 180 degrees
- renumbered BOOT1 to BOOT, RESET1 to RESET, UART1 to UART
Routing:
- net PC13: track 34.6 -> 48.2 mm, vias 1 -> 2
- net +3.3VA: track 25.7 -> 17.3 mm
- net VDC: track 165.0 -> 172.3 mm
- net +3.3V: track 53.3 -> 47.4 mm, vias 10 -> 11
- net PA10: track 17.4 -> 16.0 mm
- net /BOOT0: track 59.6 -> 58.5 mm
- net GND: track 70.7 -> 71.6 mm, vias 18 -> 19
- net SWCLK: track 63.4 -> 62.7 mm
- net PA9: track 15.2 -> 14.6 mm
Other:
- board text added: "GRUZIK 2.0"
- board text added: "S.NYDEREK 2023r"
