File: KICad_Project/Sensor/Qtr-8-SN/Qtr-8-SN.kicad_sch (KiCad schematic)
At the start: 0 parts

Commit message: 0.1
Parts:
- added C1: 0.1u, Capacitor_SMD:C_0603_1608Metric, symbol Device:C
- added C2: 1.0u, Capacitor_SMD:C_0603_1608Metric, symbol Device:C
- added IC1, IC2, IC3, IC4, IC5, IC6, IC7, IC8: ~, Sensor_Optical:KTIR0711S, symbol Sensor_KTIR0711S:KTIR0711S
- added Line_Sensor: Conn_01x11, Connector_FFC-FPC:Molex_200528-0110_1x11-1MP_P1.00mm_Horizontal, symbol Connector_Generic:Conn_01x11
- added Q1: NMOS, Package_TO_SOT_SMD:SOT-23, symbol Simulation_SPICE:NMOS
- added R1, R10, R11, R12, R13, R14, R15, R2, R3, R4, R5, R6, R7, R8, R9: 47K, Resistor_SMD:R_0603_1608Metric, symbol Device:R
Connections:
- new net: IC2.1, R1.2
- new net: IC2.4, IC4.4, IC6.4, IC8.4, R13.1, R14.1
- new net: IC4.1, R4.2
- new net: IC5.4, R7.1
- new net: IC6.1, R7.2
- new net: IC1.4, R1.1
- new net: IC3.4, R4.1
- new net: Q1.1 (D), R13.2, R14.2
- new net: IC7.4, R10.1
- new net: IC8.1, R10.2
- new net +5V: C1.1, C2.1, IC1.1, IC3.1, IC5.1, IC7.1, Line_Sensor.2 (Pin_2), R11.1, R12.1, R15.1, R2.1, R3.1, R5.1, R6.1, R8.1, R9.1
- new net GND: C1.2, C2.2, IC1.2, IC2.2, IC3.2, IC4.2, IC5.2, IC6.2, IC7.2, IC8.2, Line_Sensor.1 (Pin_1), Q1.3 (S)
- new net PA0: IC1.3, Line_Sensor.11 (Pin_11), R2.2
- new net PA1: IC2.3, Line_Sensor.10 (Pin_10), R3.2
- new net PA2: IC3.3, Line_Sensor.9 (Pin_9), R6.2
- new net PA3: IC4.3, Line_Sensor.8 (Pin_8), R5.2
- new net PA4: IC5.3, Line_Sensor.7 (Pin_7), R9.2
- new net PA5: IC6.3, Line_Sensor.6 (Pin_6), R8.2
- new net PA6: IC7.3, Line_Sensor.5 (Pin_5), R12.2
- new net PA7: IC8.3, Line_Sensor.4 (Pin_4), R11.2
- new net PB0: Line_Sensor.3 (Pin_3), Q1.2 (G), R15.2
Other:
- note added: "/TODO : Footprints / find MOSFET / Layout"
- note added: "8x KTIR0711S sensor"
- note added: "Pololu's Qtr-8x based ciruct for digital version of line sensor"
- note added: "Sensor connector"
- note added: "Supply filter"

Commit message: 0.2
Parts:
- removed Line_Sensor: Conn_01x11, Connector_FFC-FPC:Molex_200528-0110_1x11-1MP_P1.00mm_Horizontal, symbol Connector_Generic:Conn_01x11
- added C10, C3, C4, C5, C6, C7, C8, C9: 10n, Capacitor_SMD:C_0603_1608Metric, symbol Device:C
- added R16, R17: R, Resistor_THT:R_Axial_DIN0207_L6.3mm_D2.5mm_P7.62mm_Horizontal, symbol Device:R
- added Sensor(boottom_side)1: Conn_01x15, Connector_FFC-FPC:Molex_200528-0150_1x15-1MP_P1.00mm_Horizontal, symbol Connector_Generic:Conn_01x15
- Q1: footprint Package_TO_SOT_SMD:SOT-23 -> NMOS_new:NMOS_SN
- R1, R10, R4, R7: value 47K -> 48
- R11, R12, R2, R3, R5, R6, R8, R9: value 47K -> 220
- R13, R14: value 47K -> 47
Connections:
- net +5V: now also C10.2, C3.2, C4.2, C5.2, C6.2, C7.2, C8.2, C9.2, Sensor(boottom_side)1.1 (Pin_1), Sensor(boottom_side)1.2 (Pin_2), Sensor(boottom_side)1.3 (Pin_3); no longer R11.1, R12.1, R2.1, R3.1, R5.1, R6.1, R8.1, R9.1
- net GND: now also Sensor(boottom_side)1.13 (Pin_13), Sensor(boottom_side)1.14 (Pin_14), Sensor(boottom_side)1.15 (Pin_15)
- net PA0: now also R3.2, Sensor(boottom_side)1.4 (Pin_4); no longer IC1.3, R2.2
- net PA1: now also R2.2, Sensor(boottom_side)1.5 (Pin_5); no longer IC2.3, R3.2
- net PA2: now also R5.2, Sensor(boottom_side)1.6 (Pin_6); no longer IC3.3, R6.2
- net PA3: now also R6.2, Sensor(boottom_side)1.7 (Pin_7); no longer IC4.3, R5.2
- net PA4: now also R8.2, Sensor(boottom_side)1.8 (Pin_8); no longer IC5.3, R9.2
- net PA5: now also R9.2, Sensor(boottom_side)1.9 (Pin_9); no longer IC6.3, R8.2
- net PA6: now also R11.2, Sensor(boottom_side)1.10 (Pin_10); no longer IC7.3, R12.2
- net PA7: now also R12.2, Sensor(boottom_side)1.11 (Pin_11); no longer IC8.3, R11.2
- net PB0: now also Sensor(boottom_side)1.12 (Pin_12)
- new net: C4.1, IC2.3, R2.1
- new net: C3.1, IC1.3, R3.1
- new net: C5.1, IC4.3, R6.1
- new net: C8.1, IC5.3, R8.1
- new net: C6.1, IC3.3, R5.1
- new net: C7.1, IC6.3, R9.1
- new net: C9.1, IC8.3, R12.1
- new net: C10.1, IC7.3, R11.1
- no-connect marks 0 -> 4
Other:
- note added: "/TODO :check MOSFET pins / footprint + add resistors"
- note added: "Resistors"
- note removed: "/TODO : Footprints / find MOSFET / Layout"

Commit message: 0.3
Parts:
- removed Sensor(boottom_side)1: Conn_01x15, Connector_FFC-FPC:Molex_200528-0150_1x15-1MP_P1.00mm_Horizontal, symbol Connector_Generic:Conn_01x15
- added Sensor1: Conn_01x16, Connector_FFC-FPC:Molex_200528-0160_1x16-1MP_P1.00mm_Horizontal, symbol Connector_Generic:Conn_01x16
Connections:
- net +5V: now also Sensor1.13 (Pin_13), Sensor1.14 (Pin_14), Sensor1.15 (Pin_15)
- net GND: now also Sensor1.1 (Pin_1), Sensor1.2 (Pin_2), Sensor1.3 (Pin_3)
- net PA0: now also Sensor1.12 (Pin_12)
- net PA1: now also Sensor1.11 (Pin_11)
- net PA2: now also Sensor1.10 (Pin_10)
- net PA3: now also Sensor1.9 (Pin_9)
- net PA4: now also Sensor1.8 (Pin_8)
- net PA5: now also Sensor1.7 (Pin_7)
- net PA6: now also Sensor1.6 (Pin_6)
- net PA7: now also Sensor1.5 (Pin_5)
- net PB0: now also Sensor1.4 (Pin_4)
- no-connect marks 4 -> 5

Commit message: 0.5
Parts:
- R1, R10, R4, R7: value 48 -> 39
Other:
- note removed: "/TODO :check MOSFET pins / footprint + add resistors"
Changed lines of the file:
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@@
     (fill (type none))
-  )
-  (text "/TODO :check MOSFET pins / footprint + add resistors "
-    (at 111.76 59.69 0)
-    (effects (font (size 1.27 1.27)) (justify left bottom))
   )
   (text "Sensor connector" (at 16.51 17.78 0)
@@
       (effects (font (size 1.27 1.27)) (justify left))
     )
-    (property "Value" "48" (at 54.61 86.36 0)
+    (property "Value" "39" (at 54.61 86.36 0)
       (effects (font (size 1.27 1.27)) (justify left))
     )
@@
       (effects (font (size 1.27 1.27)) (justify left))
     )
-    (property "Value" "48" (at 87.63 86.36 0)
+    (property "Value" "39" (at 87.63 86.36 0)
       (effects (font (size 1.27 1.27)) (justify left))
     )
@@
       (effects (font (size 1.27 1.27)) (justify left))
     )
-    (property "Value" "48" (at 21.59 86.36 0)
+    (property "Value" "39" (at 21.59 86.36 0)
       (effects (font (size 1.27 1.27)) (justify left))
     )
@@
       (effects (font (size 1.27 1.27)) (justify left))
     )
-    (property "Value" "48" (at 120.65 87.63 0)
-      (effects (font (size 1.27 1.27)) (justify left))
-    )
+    (property "Value" "39" (at 120.65 87.63 0)
+      (effects (font (size 1.27 1.27)) (justify left))
+    )
