File: KICad_Project/Sensor/Qtr-8-SN/Qtr-8-SN.kicad_pcb (KiCad board)
At the start: 2 copper layers, 84.7 x 22.3 mm, 39 parts, among them Q1 NMOS

Commit message: 0.3
Parts:
- removed Sensor(boottom_side)1: Conn_01x15, Connector_FFC-FPC:Molex_200528-0150_1x15-1MP_P1.00mm_Horizontal
- added Sensor1: Conn_01x16, Connector_FFC-FPC:Molex_200528-0160_1x16-1MP_P1.00mm_Horizontal, B.Cu at (93.8, 141.9)
- moved C2 1.29 mm to (108.0, 143.1)
- moved C1 1.29 mm to (108.1, 144.8)
- moved R9 0.46 mm to (81.3, 138.5)
- moved R5 0.43 mm to (109.8, 138.5)

Commit message: 0.5
Parts:
- R1, R10, R4, R7: value 48 -> 39
- moved R15 7.47 mm to (79.4, 144.8)
- moved R6 2.14 mm to (98.2, 138.3)
- moved R5 1.79 mm to (108.0, 138.4)
- moved R8 1.68 mm to (89.2, 138.4)
- moved C6 0.31 mm to (110.5, 136.6)
- moved C10 0.26 mm to (72.5, 136.4)
- moved R2 0.23 mm to (119.3, 138.6)
- moved C5 0.20 mm to (101.1, 136.4)
- moved R9 0.16 mm to (81.1, 138.6)
- moved C8 0.15 mm to (91.5, 136.4)
- turned C1 to 180 degrees
- renumbered Sensor1 to Sensor
Routing:
- net Net-(IC2-Pad4): track 0.00 -> 82.0 mm, vias 0 -> 4
- net PA7: track 0.00 -> 43.0 mm, vias 0 -> 2
- net PA0: track 0.00 -> 40.9 mm, vias 0 -> 2
- net PA1: track 0.00 -> 32.0 mm, vias 0 -> 2
- net PA6: track 0.00 -> 31.5 mm
- net PB0: track 0.00 -> 26.3 mm
- net +5V: track 0.00 -> 22.7 mm, vias 0 -> 15
- net PA5: track 0.00 -> 20.0 mm
- net PA2: track 0.00 -> 19.2 mm, vias 0 -> 2
- net Net-(Q1-D): track 0.00 -> 13.6 mm
- net Net-(IC7-Pad4): track 0.00 -> 8.85 mm
- net Net-(IC1-Pad4): track 0.00 -> 8.81 mm
- net Net-(IC5-Pad4): track 0.00 -> 8.77 mm
- net Net-(IC3-Pad4): track 0.00 -> 8.62 mm
- net Net-(IC8-Pad1): track 0.00 -> 8.35 mm
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- added copper zone on F.Cu, net +5V
- added copper zone on B.Cu, net GND
Other:
- board size 84.7 x 22.3 mm -> 84.7 x 23.3 mm
- board text added: "GRUZIK2.0"

Commit message: 0.6
Parts:
- moved R12 2.70 mm to (64.9, 138.9)
- moved REF** 2.34 mm to (117.8, 146.8)
- moved REF** 2.34 mm to (67.5, 146.8)
Routing:
- net PA7: track 43.0 -> 40.8 mm
- net Net-(C9-Pad1): track 4.81 -> 6.87 mm
- net PA0: track 40.9 -> 40.2 mm
Other:
- outline, holes or cut-outs redrawn
Changed lines of the file:
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@@
   (net 34 "unconnected-(Sensor1-Pin_16-Pad16)")
   (footprint "MountingHole:MountingHole_2.1mm" (layer "F.Cu")
-    (at 120.1136 146.7956)
+    (at 117.7761 146.7956)
     (descr "Mounting Hole 2.1mm, no annular")
     (tags "mounting hole 2.1mm no annular")
@@
   )
   (footprint "MountingHole:MountingHole_2.1mm" (layer "F.Cu")
-    (at 65.1466 146.7956)
+    (at 67.4841 146.7956)
     (descr "Mounting Hole 2.1mm, no annular")
     (tags "mounting hole 2.1mm no annular")
@@
     (property "ki_keywords" "R res resistor")
     (attr smd)
-    (fp_text reference "R3" (at 1.5748 -1.3716) (layer "B.SilkS")
+    (fp_text reference "R3" (at 1.3208 1.3716) (layer "B.SilkS")
         (effects (font (size 1 1) (thickness 0.2) bold) (justify mirror))
     )
@@
   )
   (footprint "Resistor_SMD:R_0603_1608Metric" (layer "B.Cu")
-    (at 62.1792 139.0396 -90)
+    (at 64.8716 138.875 -90)
     (descr "Resistor SMD 0603 (1608 Metric), square (rectangular) end terminal, IPC_7351 nominal, (Body size source: IPC-SM-782 page 72, https://www.pcb-3d.com/wordpress/wp-content/uploads/ipc-sm-782a_amendment_1_and_2.pdf), generated with kicad-footprint-generator")
     (tags "resistor")
@@
     (property "ki_keywords" "R res resistor")
     (attr smd)
-    (fp_text reference "R12" (at -0.508 1.4732 90) (layer "B.SilkS")
+    (fp_text reference "R12" (at -0.0894 1.4224 90) (layer "B.SilkS")
         (effects (font (size 1 1) (thickness 0.2) bold) (justify mirror))
     )
@@
   (gr_line (start 134.9676 132.7956) (end 134.9676 138.7956)
     (stroke (width 0.15) (type default)) (layer "Edge.Cuts"))
-  (gr_arc (start 123.6136 143.2956) (mid 124.638726 140.820727) (end 127.1136 139.7956)
+  (gr_arc (start 121.2761 143.2956) (mid 122.301226 140.820727) (end 124.7761 139.7956)
+    (stroke (width 0.15) (type default)) (layer "Edge.Cuts"))
+  (gr_line (start 60.4841 139.7956) (end 58.1466 139.7956)
     (stroke (width 0.15) (type default)) (layer "Edge.Cuts"))
   (gr_arc (start 134.9676 138.7956) (mid 134.674707 139.502707) (end 133.9676 139.7956)
     (stroke (width 0.15) (type default)) (layer "Edge.Cuts"))
-  (gr_line (start 61.6466 146.7956) (end 61.6466 143.2956)
+  (gr_line (start 63.9841 146.7956) (end 63.9841 143.2956)
     (stroke (width 0.15) (type default)) (layer "Edge.Cuts"))
-  (gr_arc (start 58.1466 139.7956) (mid 60.621473 140.820726) (end 61.6466 143.2956)
+  (gr_line (start 127.1136 139.7956) (end 124.7761 139.7956)
+    (stroke (width 0.15) (type default)) (layer "Edge.Cuts"))
+  (gr_arc (start 60.4841 139.7956) (mid 62.958973 140.820726) (end 63.9841 143.2956)
     (stroke (width 0.15) (type default)) (layer "Edge.Cuts"))
   (gr_line (start 134.9676 127.9712) (end 134.9676 132.7956)
     (stroke (width 0.15) (type default)) (layer "Edge.Cuts"))
-  (gr_arc (start 68.6466 146.7956) (mid 65.1466 150.2956) (end 61.6466 146.7956)
+  (gr_arc (start 70.9841 146.7956) (mid 67.4841 150.2956) (end 63.9841 146.7956)
     (stroke (width 0.15) (type default)) (layer "Edge.Cuts"))
-  (gr_line (start 116.6136 146.7956) (end 68.6466 146.7956)
+  (gr_line (start 114.2761 146.7956) (end 70.9841 146.7956)
     (stroke (width 0.15) (type default)) (layer "Edge.Cuts"))
   (gr_line (start 50.2926 132.8056) (end 50.2926 138.8056)
     (stroke (width 0.15) (type default)) (layer "Edge.Cuts"))
-  (gr_line (start 123.6136 146.7956) (end 123.6136 143.2956)
+  (gr_line (start 121.2761 146.7956) (end 121.2761 143.2956)
     (stroke (width 0.15) (type default)) (layer "Edge.Cuts"))
   (gr_arc (start 133.9676 126.9712) (mid 134.674706 127.264093) (end 134.9676 127.9712)
@@
   (gr_line (start 58.1466 139.7956) (end 51.2926 139.8056)
     (stroke (width 0.15) (type default)) (layer "Edge.Cuts"))
-  (gr_arc (start 123.6136 146.7956) (mid 120.1136 150.2956) (end 116.6136 146.7956)
+  (gr_arc (start 121.2761 146.7956) (mid 117.7761 150.2956) (end 114.2761 146.7956)
     (stroke (width 0.15) (type default)) (layer "Edge.Cuts"))
   (gr_line (start 125.9676 132.7956) (end 134.9676 132.7956)
@@
   (segment (start 90.5378 137.5542) (end 90.7666 137.3254) (width 0.3) (layer "B.Cu") (net 8))
   (segment (start 90.0176 134.5692) (end 90.7796 135.3312) (width 0.3) (layer "B.Cu") (net 8))
+  (segment (start 62.866 138.05) (end 62.23 137.414) (width 0.25) (layer "B.Cu") (net 9))
   (segment (start 62.1792 135.1788) (end 62.1792 136.3472) (width 0.3) (layer "B.Cu") (net 9))
   (segment (start 61.4426 134.4422) (end 62.1792 135.1788) (width 0.3) (layer "B.Cu") (net 9))
-  (segment (start 62.1792 136.3472) (end 62.1792 138.2146) (width 0.3) (layer "B.Cu") (net 9))
+  (segment (start 64.8716 138.05) (end 62.866 138.05) (width 0.25) (layer "B.Cu") (net 9))
+  (segment (start 62.23 137.414) (end 62.23 136.398) (width 0.25) (layer "B.Cu") (net 9))
   (segment (start 61.4426 133.7056) (end 61.4426 134.4422) (width 0.3) (layer "B.Cu") (net 9))
   (segment (start 71.6788 135.2804) (end 71.6788 136.1948) (width 0.3) (layer "B.Cu") (net 10))
@@
   (segment (start 117.2972 139.7) (end 118.0084 139.7) (width 0.3) (layer "B.Cu") (net 22))
   (segment (start 118.0084 139.7) (end 118.2116 139.4968) (width 0.3) (layer "B.Cu") (net 22))
+  (segment (start 117.9068 142.2908) (end 116.9336 141.3176) (width 0.3) (layer "F.Cu") (net 23))
+  (segment (start 119.1768 142.2908) (end 117.9068 142.2908) (width 0.3) (layer "F.Cu") (net 23))
+  (segment (start 116.9336 141.3176) (end 98.306 141.3176) (width 0.3) (layer "F.Cu") (net 23))
+  (segment (start 97.5868 143.256) (end 96.8328 144.01) (width 0.3) (layer "F.Cu") (net 23))
   (segment (start 98.306 141.3176) (end 97.5868 142.0368) (width 0.3) (layer "F.Cu") (net 23))
-  (segment (start 116.9336 141.3176) (end 98.306 141.3176) (width 0.3) (layer "F.Cu") (net 23))
+  (segment (start 96.8328 144.01) (end 91.9908 144.01) (width 0.3) (layer "F.Cu") (net 23))
+  (segment (start 97.5868 142.0368) (end 97.5868 143.256) (width 0.3) (layer "F.Cu") (net 23))
   (segment (start 91.9908 144.01) (end 91.0844 143.1036) (width 0.3) (layer "F.Cu") (net 23))
-  (segment (start 96.8328 144.01) (end 91.9908 144.01) (width 0.3) (layer "F.Cu") (net 23))
-  (segment (start 97.5868 143.256) (end 96.8328 144.01) (width 0.3) (layer "F.Cu") (net 23))
-  (segment (start 117.9068 142.2908) (end 116.9336 141.3176) (width 0.3) (layer "F.Cu") (net 23))
-  (segment (start 119.6848 142.2908) (end 117.9068 142.2908) (width 0.3) (layer "F.Cu") (net 23))
-  (segment (start 97.5868 142.0368) (end 97.5868 143.256) (width 0.3) (layer "F.Cu") (net 23))
   (via (at 91.0844 143.1036) (size 0.55) (drill 0.25) (layers "F.Cu" "B.Cu") (net 23))
-  (via (at 119.6848 142.2908) (size 0.55) (drill 0.25) (layers "F.Cu" "B.Cu") (net 23))
-  (segment (start 120.904 142.2908) (end 122.5804 140.6144) (width 0.3) (layer "B.Cu") (net 23))
+  (via (at 119.1768 142.2908) (size 0.55) (drill 0.25) (layers "F.Cu" "B.Cu") (net 23))
+  (segment (start 119.1768 142.2908) (end 119.5832 142.2908) (width 0.3) (layer "B.Cu") (net 23))
   (segment (start 90.2556 140.97) (end 90.2556 142.2748) (width 0.3) (layer "B.Cu") (net 23))
+  (segment (start 119.5832 142.2908) (end 123.3424 138.5316) (width 0.3) (layer "B.Cu") (net 23))
+  (segment (start 90.2556 142.2748) (end 91.0844 143.1036) (width 0.3) (layer "B.Cu") (net 23))
   (segment (start 123.3424 138.5316) (end 124.6002 138.5316) (width 0.3) (layer "B.Cu") (net 23))
-  (segment (start 119.6848 142.2908) (end 120.904 142.2908) (width 0.3) (layer "B.Cu") (net 23))
-  (segment (start 122.5804 139.2936) (end 123.3424 138.5316) (width 0.3) (layer "B.Cu") (net 23))
-  (segment (start 90.2556 142.2748) (end 91.0844 143.1036) (width 0.3) (layer "B.Cu") (net 23))
-  (segment (start 122.5804 140.6144) (end 122.5804 139.2936) (width 0.3) (layer "B.Cu") (net 23))
   (segment (start 67.056 142.5448) (end 68.7324 142.5448) (width 0.3) (layer "F.Cu") (net 24))
   (via (at 68.7324 142.5448) (size 0.55) (drill 0.25) (layers "F.Cu" "B.Cu") (net 24))
   (via (at 67.056 142.5448) (size 0.55) (drill 0.25) (layers "F.Cu" "B.Cu") (net 24))
-  (segment (start 62.738 142.1384) (end 63.1444 142.5448) (width 0.3) (layer "B.Cu") (net 24))
+  (segment (start 64.8716 139.7) (end 64.8716 140.6144) (width 0.25) (layer "B.Cu") (net 24))
   (segment (start 68.7324 142.5448) (end 81.026 142.5448) (width 0.3) (layer "B.Cu") (net 24))
+  (segment (start 65.1764 140.9192) (end 66.8528 140.9192) (width 0.25) (layer "B.Cu") (net 24))
   (segment (start 81.3816 144.526) (end 81.9404 145.0848) (width 0.3) (layer "B.Cu") (net 24))
   (segment (start 81.9404 145.0848) (end 96.774 145.0848) (width 0.3) (layer "B.Cu") (net 24))
   (segment (start 81.026 142.5448) (end 81.3816 142.9004) (width 0.3) (layer "B.Cu") (net 24))
   (segment (start 96.774 145.0848) (end 97.2556 144.6032) (width 0.3) (layer "B.Cu") (net 24))
-  (segment (start 62.1792 141.5796) (end 62.738 142.1384) (width 0.3) (layer "B.Cu") (net 24))
-  (segment (start 62.1792 139.8646) (end 62.1792 141.5796) (width 0.3) (layer "B.Cu") (net 24))
+  (segment (start 67.056 141.1224) (end 67.056 142.5448) (width 0.25) (layer "B.Cu") (net 24))
   (segment (start 97.2556 144.6032) (end 97.2556 140.97) (width 0.3) (layer "B.Cu") (net 24))
-  (segment (start 63.1444 142.5448) (end 67.056 142.5448) (width 0.3) (layer "B.Cu") (net 24))
   (segment (start 81.3816 142.9004) (end 81.3816 144.526) (width 0.3) (layer "B.Cu") (net 24))
+  (segment (start 66.8528 140.9192) (end 67.056 141.1224) (width 0.25) (layer "B.Cu") (net 24))
+  (segment (start 64.8716 140.6144) (end 65.1764 140.9192) (width 0.25) (layer "B.Cu") (net 24))
   (segment (start 81.8896 142.4432) (end 84.5788 142.4432) (width 0.3) (layer "B.Cu") (net 25))
   (segment (start 81.28 141.8336) (end 81.8896 142.4432) (width 0.3) (layer "B.Cu") (net 25))
