File: Gruzik2.0-light/PCB/KICad_Project/Gruzik2.0/Gruzik2.0.kicad_pcb (KiCad board)
At the start: 4 copper layers, 128 x 39.9 mm, 56 parts, among them U1 STM32F103C8T6, U2 LM1117MP-3.3, U3 LM1117MP-5.0, U3V40F7-POLOLU Conn_01x06, U4 TB6612FNG, U5 TB6612FNG, U7 HC-05, Y1 8MHz

Commit message: 9.0
Parts:
- renumbered Motor-Battery_L1 to Motor-Battery_L, Motor-Battery_R1 to Motor-Battery_R, Motor-STAB-Battery-L1 to Motor-STAB-Battery-L, Motor-STAB-Battery-R1 to Motor-STAB-Battery-R
Changed lines of the file:
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@@
     (property "ki_keywords" "solder jumper SPST")
     (attr exclude_from_pos_files)
-    (fp_text reference "Motor-STAB-Battery-R1" (at 11.1356 -0.4064) (layer "F.SilkS")
+    (fp_text reference "Motor-STAB-Battery-R" (at 11.1356 -0.4064) (layer "F.SilkS")
         (effects (font (size 1 1) (thickness 0.2) bold))
     )
@@
     (property "ki_keywords" "solder jumper SPST")
     (attr exclude_from_pos_files)
-    (fp_text reference "Motor-Battery_R1" (at -8.494 0.254) (layer "F.SilkS")
+    (fp_text reference "Motor-Battery_R" (at -8.494 0.254) (layer "F.SilkS")
         (effects (font (size 1 1) (thickness 0.2) bold))
     )
@@
     (property "ki_keywords" "solder jumper SPST")
     (attr exclude_from_pos_files)
-    (fp_text reference "Motor-STAB-Battery-L1" (at 10.9116 0.762) (layer "F.SilkS")
+    (fp_text reference "Motor-STAB-Battery-L" (at 10.9116 0.762) (layer "F.SilkS")
         (effects (font (size 1 1) (thickness 0.2) bold))
     )
@@
     (property "ki_keywords" "solder jumper SPST")
     (attr exclude_from_pos_files)
-    (fp_text reference "Motor-Battery_L1" (at -8.2192 -0.1016) (layer "F.SilkS")
+    (fp_text reference "Motor-Battery_L" (at -8.2192 -0.1016) (layer "F.SilkS")
         (effects (font (size 1 1) (thickness 0.2) bold))
     )
