File: Gruzik2.0-light/PCB/KICad_Project/Gruzik2.0/Gruzik2.0.kicad_sch (KiCad schematic)
At the start: 47 parts, among them U1 STM32F103C8T6, U2 LM1117MP-3.3, U3 LM1117MP-5.0, U3V40F7-POLOLU1 Conn_01x06, U3V40F7-POLOLU2 Conn_01x06, U4 TB6612FNG, U5 TB6612FNG, U7 HC-05, Y1 8MHz

Commit message: 9.0
Other:
- note removed: "TODO: footprint of polarized capacitors / figure out how to mount cleaners for wheels"
Changed lines of the file:
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@@
-    (effects (font (size 2.0066 2.0066) (thickness 0.4013) bold) (justify left bottom))
-  )
-  (text "TODO: footprint of polarized capacitors / figure out how to mount cleaners for wheels"
-    (at 273.05 250.19 0)
     (effects (font (size 2.0066 2.0066) (thickness 0.4013) bold) (justify left bottom))
   )
